File: PCB/USB-Hub.kicad_pcb (KiCad board)
At the start: 2 copper layers, 60 x 38 mm, 29 parts, among them U1 SL2.1S, U2 USBLC6-2SC6-ES, U3 USBLC6-2SC6-ES, U4 USBLC6-2SC6-ES

Commit message: update
Parts:
- moved R1 1.10 mm to (81.2, 56.1)
Connections:
- U2 pad 1: /D- -> unconnected-(U2-I/O1-Pad1)
- U2 pad 4: unconnected-(U2-I/O2-Pad4) -> /D-
Routing:
- net /D-: track 29.4 -> 52.4 mm, vias 0 -> 2
- net /D+: track 40.7 -> 57.6 mm
- net /D3-: track 35.0 -> 38.4 mm
- net /D3+: track 44.9 -> 47.2 mm
- net +5V: track 154.2 -> 155.9 mm
- net Net-(USB1-CC1): track 2.63 -> 3.77 mm
- net /D4+: track 41.9 -> 42.7 mm
