File: PCB/USB-Hub.kicad_sch (KiCad schematic)
At the start: 29 parts, among them U1 SL2.1S, U2 USBLC6-2SC6-ES, U3 USBLC6-2SC6-ES, U4 USBLC6-2SC6-ES

Commit message: update
Connections:
- net D-: now also U2.4 (I/O2); no longer U2.1 (I/O1)
Changed lines of the file:
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@@
-	)
-	(no_connect
-		(at 57.15 99.06)
 	)
 	(no_connect
@@
 	)
 	(no_connect
+		(at 26.67 81.28)
+	)
+	(no_connect
 		(at 257.81 90.17)
 	)
@@
 	(wire
 		(pts
+			(xy 57.15 99.06) (xy 60.96 99.06)
+		)
+		(stroke
+			(width 0)
+			(type default)
+		)
+	)
+	(wire
+		(pts
 			(xy 255.27 69.85) (xy 257.81 69.85)
 		)
@@
 		(pts
 			(xy 248.92 45.72) (xy 228.6 45.72)
-		)
-		(stroke
-			(width 0)
-			(type default)
-		)
-	)
-	(wire
-		(pts
-			(xy 22.86 81.28) (xy 26.67 81.28)
 		)
 		(stroke
@@
 		)
 	)
-	(label "D-"
-		(at 25.4 81.28 180)
-		(effects
-			(font
-				(size 1.27 1.27)
-			)
-			(justify right bottom)
-		)
-	)
 	(label "D3-"
 		(at 251.46 36.83 0)
@@
 		)
 	)
+	(label "D-"
+		(at 60.96 99.06 180)
+		(effects
+			(font
+				(size 1.27 1.27)
+			)
+			(justify right bottom)
+		)
+	)
